Commit message: v0.6

File: urdf_sdf/model/element.xacro (robot description, xacro)
@@ -49,5 +49,5 @@
 		<parent link="${element_name}_1"/>
 		<child  link="${element_name}_2"/>
-		<origin xyz="0 ${-height} 0" rpy="-1.57 0 0"/>
+		<origin xyz="0 ${-height} 0" rpy="${-pi/2} 0 0"/>
     </joint>
     <!-- 3 to 2 -->
@@ -56,5 +56,5 @@
 		<parent link="${element_name}_2"/>
 		<child  link="${element_name}_3"/>
-		<origin xyz="0 ${-height} 0" rpy="-1.57 0 0"/>
+		<origin xyz="0 ${-height} 0" rpy="${-pi/2} 0 0"/>
     </joint>
     <!-- 4 to 3 -->
@@ -63,5 +63,5 @@
 		<parent link="${element_name}_3"/>
 		<child  link="${element_name}_4"/>
-		<origin xyz="0 ${-height} 0" rpy="-1.57 0 0"/>
+		<origin xyz="0 ${-height} 0" rpy="${-pi/2} 0 0"/>
     </joint>
     <!-- 1 to 4: Close the loop by injection of SDF-code into UDRF -->
