Commit message: v0.5

File: model/element.xacro (robot description, xacro)
@@ -4,29 +4,29 @@
     <!-- Macro for a single element of box geometry -->
     <xacro:macro name="elem" params="element_number element_colour:=White">
-		<!-- Link without joint -->
-		<link name="${element_name}_${element_number}">
-			<visual>
-				<geometry>
-					<box size="${width} ${height} ${thickness}"/>
-				</geometry>
-				<origin xyz="0 ${-height/2} 0" rpy="0 0 0"/>
-			</visual>
-			<collision>
-				<geometry>
-					<box size="${width} ${height} ${thickness}"/>
-				</geometry>
-				<origin xyz="0 ${-height/2} 0" rpy="0 0 0"/>
-			</collision>
-			<xacro:box_inertial m="${mass}"
-			                    x="0"          y="${-height/2}"  z="0"
-			                    dx="${width}" dy="${height}"    dz="${thickness}"/>
-		</link>
-		<!-- Gazebo simulation settings -->
-		<gazebo reference="${element_name}_${element_number}">
-			<selfCollide>true</selfCollide>
-			<static>false</static>
-			<turnGravityOff>false</turnGravityOff>
-			<material>Gazebo/${element_colour}</material>
-		</gazebo>
+        <!-- Link without joint -->
+        <link name="${element_name}_${element_number}">
+            <visual>
+                <geometry>
+                    <box size="${width} ${height} ${thickness}"/>
+                </geometry>
+                <origin xyz="0 ${-height/2} 0" rpy="0 0 0"/>
+            </visual>
+            <collision>
+                <geometry>
+                    <box size="${width} ${height} ${thickness}"/>
+                </geometry>
+                <origin xyz="0 ${-height/2} 0" rpy="0 0 0"/>
+            </collision>
+            <xacro:box_inertial m="${mass}"
+                                x="0"          y="${-height/2}"  z="0"
+                                dx="${width}" dy="${height}"    dz="${thickness}"/>
+        </link>
+        <!-- Gazebo simulation settings -->
+        <gazebo reference="${element_name}_${element_number}">
+            <selfCollide>true</selfCollide>
+            <static>false</static>
+            <turnGravityOff>false</turnGravityOff>
+            <material>Gazebo/${element_colour}</material>
+        </gazebo>
     </xacro:macro>
     <!-- Fixed world frame -->
@@ -40,28 +40,28 @@
     <!-- 1 to world -->
     <joint name="1_to_world" type="fixed">
-		<parent link="world"/>
-		<child  link="${element_name}_1"/>
-		<origin xyz="0 ${height/2} 1" rpy="0 0 0"/>
+        <parent link="world"/>
+        <child  link="${element_name}_1"/>
+        <origin xyz="0 ${height/2} 1" rpy="0 0 0"/>
     </joint>
     <!-- 2 to 1 -->
     <joint name="2_to_1" type="continuous">
-		<axis xyz="1 0 0"/>
-		<parent link="${element_name}_1"/>
-		<child  link="${element_name}_2"/>
-		<origin xyz="0 ${-height} 0" rpy="${-pi/2} 0 0"/>
+        <axis xyz="1 0 0"/>
+        <parent link="${element_name}_1"/>
+        <child  link="${element_name}_2"/>
+        <origin xyz="0 ${-height} 0" rpy="${-pi/2} 0 0"/>
     </joint>
     <!-- 3 to 2 -->
     <joint name="3_to_2" type="continuous">
-		<axis xyz="1 0 0"/>
-		<parent link="${element_name}_2"/>
-		<child  link="${element_name}_3"/>
-		<origin xyz="0 ${-height} 0" rpy="${-pi/2} 0 0"/>
+        <axis xyz="1 0 0"/>
+        <parent link="${element_name}_2"/>
+        <child  link="${element_name}_3"/>
+        <origin xyz="0 ${-height} 0" rpy="${-pi/2} 0 0"/>
     </joint>
     <!-- 4 to 3 -->
     <joint name="4_to_3" type="continuous">
-		<axis xyz="1 0 0"/>
-		<parent link="${element_name}_3"/>
-		<child  link="${element_name}_4"/>
-		<origin xyz="0 ${-height} 0" rpy="${-pi/2} 0 0"/>
+        <axis xyz="1 0 0"/>
+        <parent link="${element_name}_3"/>
+        <child  link="${element_name}_4"/>
+        <origin xyz="0 ${-height} 0" rpy="${-pi/2} 0 0"/>
     </joint>
     <!-- 1 to 4: Close the loop by injection of SDF-code into UDRF -->
@@ -72,19 +72,19 @@
     <gazebo>
         <joint name='1_to_4' type='revolute'>
-		  <child>${element_name}_1</child>
-		  <parent>${element_name}_4</parent>
-		  <axis>
-			<xyz>1 0 0</xyz>
-			<limit>
-			  <lower>-1e+16</lower>
-			  <upper>1e+16</upper>
-			</limit>
-			<dynamics>
-			  <spring_reference>0</spring_reference>
-			  <spring_stiffness>0</spring_stiffness>
-			</dynamics>
-			<use_parent_model_frame>1</use_parent_model_frame>
-		  </axis>
-		</joint>
+            <child>${element_name}_1</child>
+            <parent>${element_name}_4</parent>
+            <axis>
+                <xyz>1 0 0</xyz>
+                <limit>
+                    <lower>-1e+16</lower>
+                    <upper>1e+16</upper>
+                </limit>
+                <dynamics>
+                    <spring_reference>0</spring_reference>
+                    <spring_stiffness>0</spring_stiffness>
+                </dynamics>
+                <use_parent_model_frame>1</use_parent_model_frame>
+            </axis>
+        </joint>
     </gazebo>
 </robot>

Commit message: v0.5

File: model/element.xacro (robot description, xacro)
@@ -39,5 +39,5 @@
     <!-- Joints -->
     <!-- 1 to world -->
-    <joint name="1_to_world" type="fixed">
+    <joint name="1_to_world" type="floating">
         <parent link="world"/>
         <child  link="${element_name}_1"/>

Commit message: feat: Added Docker and Docker-Compose files, separated documentation and fixed the robot in space again

File: model/element.xacro (robot description, xacro)
@@ -39,8 +39,8 @@
     <!-- Joints -->
     <!-- 1 to world -->
-    <joint name="1_to_world" type="floating">
+    <joint name="1_to_world" type="fixed">
         <parent link="world"/>
         <child  link="${element_name}_1"/>
-        <origin xyz="0 ${height/2} 1" rpy="0 0 0"/>
+        <origin xyz="0 ${height/2} ${height/2}" rpy="0 0 0"/>
     </joint>
     <!-- 2 to 1 -->
