Commit message: core: Upgraded code to ROS2

File: urdf/element.xacro (robot description, xacro)
@@ -1,7 +1,6 @@
 <?xml version="1.0"?>
-<robot
-    xmlns:xacro="http://www.ros.org/wiki/xacro" name="element">
+<robot xmlns:xacro="http://www.ros.org/wiki/xacro" name="element">
     <!-- Macro for a single element of box geometry -->
-    <xacro:macro name="elem" params="element_number element_colour:=White">
+    <xacro:macro name="elem" params="element_number is_gravity:=false element_colour:=White">
         <!-- Link without joint -->
         <link name="${element_name}_${element_number}">
@@ -26,5 +25,5 @@
             <selfCollide>true</selfCollide>
             <static>false</static>
-            <turnGravityOff>false</turnGravityOff>
+            <turnGravityOff>${not is_gravity}</turnGravityOff>
             <material>Gazebo/${element_colour}</material>
         </gazebo>
@@ -33,8 +32,8 @@
     <link name="world"/>
     <!-- Elements without joints -->
-    <xacro:elem element_number="1" element_colour="Red"   />
-    <xacro:elem element_number="2" element_colour="Green" />
-    <xacro:elem element_number="3" element_colour="Blue"  />
-    <xacro:elem element_number="4" element_colour="Yellow"/>
+    <xacro:elem element_number="1" is_gravity="$(arg is_gravity)" element_colour="Red"/>
+    <xacro:elem element_number="2" is_gravity="$(arg is_gravity)" element_colour="Green"/>
+    <xacro:elem element_number="3" is_gravity="$(arg is_gravity)" element_colour="Blue"/>
+    <xacro:elem element_number="4" is_gravity="$(arg is_gravity)" element_colour="Yellow"/>
     <!-- Joints -->
     <!-- 1 to world -->
@@ -65,5 +64,5 @@
         <origin xyz="0 ${-height} 0" rpy="${-pi/2} 0 0"/>
     </joint>
-    <!-- 1 to 4: Close the loop by injection of SDF-code into UDRF -->
+    <!-- 1 to 4 - Close the loop by injection of SDF-code into UDRF -->
     <!-- You can even use macro syntax ${} here as illustraded by the
          the variable ${element_name}. -->

File: urdf/parameters.xacro (robot description, xacro)
@@ -1,5 +1,4 @@
 <?xml version="1.0"?>
-<robot
-    xmlns:xacro="http://www.ros.org/wiki/xacro" >
+<robot xmlns:xacro="http://www.ros.org/wiki/xacro" >
     <!-- Box geometry -->
     <xacro:property name="element_name" value="element"/>
@@ -8,4 +7,5 @@
     <xacro:property name="thickness"    value="0.1"/>
     <xacro:property name="mass"         value="5.0"/>
+    <xacro:arg name="is_gravity" default="true"/>
     <!-- Macro for inertia matrix for rectangular box around its center -->
     <xacro:macro name="box_inertial" params="m x y z dx dy dz">
